File: boards/Tadpole - Breadboard/Rev1.0.sch (EAGLE design)
At the start: 0 parts

Commit message: Final rev 1.0 brain and initial tadpole breadboard.
Parts:
- added JP1, JP2, JP3, JP4, JP5, JP6, JP7, JP8: HEADER-1X8, lib-works:HEADER-1X8
Connections:
- new net FLASHSEL: JP3.8, JP7.8
- new net GND: JP3.1, JP3.2, JP3.3, JP4.3, JP4.4, JP4.8, JP7.1, JP7.2, JP7.3, JP8.3, JP8.4, JP8.8
- new net ICSPCLK: JP2.7, JP6.7
- new net ICSPDAT: JP2.8, JP6.8
- new net RA0: JP1.1, JP5.1
- new net RA1: JP1.2, JP5.2
- new net RA2: JP1.3, JP5.3
- new net RA3: JP1.4, JP5.4
- new net RA4: JP1.5, JP5.5
- new net RA5: JP1.6, JP5.6
- new net RA6: JP1.7, JP5.7
- new net RA7: JP1.8, JP5.8
- new net RB0: JP2.1, JP6.1
- new net RB1: JP2.2, JP6.2
- new net RB2: JP2.3, JP6.3
- new net RB3: JP2.4, JP6.4
- new net RB4: JP2.5, JP6.5
- new net RB5: JP2.6, JP6.6
- new net RC5: JP3.6, JP7.6
- new net RC6: JP3.7, JP7.7
- new net SCK: JP4.7, JP8.7
- new net SI: JP4.5, JP8.5
- new net SO: JP4.6, JP8.6
- new net UARTRX: JP3.4, JP7.4
- new net UARTTX: JP3.5, JP7.5
- new net VDD: JP4.2, JP8.2
- new net VIN: JP4.1, JP8.1
