File: boards/dAuratus/dAratus.kicad_pcb (KiCad board)
At the start: 2 copper layers, 40 x 35 mm, 21 parts, among them J1 Conn_01x03_Male, J2 Conn_01x08_Female, J3 Conn_01x08_Female, J4 Conn_01x08_Female, J5 Conn_01x02_Male, SW1 SW_SPDT, U1 ADP7104ARDZ, U2 AVR128DB28-SOIC, U3 AT25xxx

Commit message: Huge update, long overdue.
Parts:
- added G***: LOGO, lib:eFrog-pcb, F.Cu at (103.5, 117.5)
Other:
- board text added: "/MSS"
- board text added: "MISO"
- board text added: "MOSI"
- board text added: "PD1"
- board text added: "PD7"
- board text added: "SCK"
- board text added: "dAuratus v1.0"
- board text removed: "PA1"
- board text removed: "PA2"
- board text removed: "PA3"
- board text removed: "PA4"
- board text removed: "PA5"
- board text removed: "PA6"
- board text removed: "dAuratus"
